Commit message: add mesh ref to urdf

File: ros2/urdf/miranda.urdf (robot description, URDF)
Before this commit: robot miranda, 17 links, 16 joints
Links:
- link J1_A_stator: geometry collision mesh filename=package://concert_resources/models/modular/meshes/concert/s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 scale=0.001 0.001 0.001; visual mesh filename=package://concert_resources/models/modular/meshes/concert/c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 scale=0.001 0.001 0.001
- link J2_A_stator: geometry collision mesh filename=package://concert_resources/models/modular/meshes/concert/s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 scale=0.001 0.001 0.001; visual mesh filename=package://concert_resources/models/modular/meshes/concert/c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 scale=0.001 0.001 0.001
- link J3_A_stator: geometry collision mesh filename=package://concert_resources/models/modular/meshes/concert/s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 scale=0.001 0.001 0.001; visual mesh filename=package://concert_resources/models/modular/meshes/concert/c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 scale=0.001 0.001 0.001
- link J4_A_stator: geometry collision mesh filename=package://concert_resources/models/modular/meshes/concert/s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 scale=0.001 0.001 0.001; visual mesh filename=package://concert_resources/models/modular/meshes/concert/c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 scale=0.001 0.001 0.001
- link J5_A_stator: geometry collision mesh filename=package://concert_resources/models/modular/meshes/concert/s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 scale=0.001 0.001 0.001; visual mesh filename=package://concert_resources/models/modular/meshes/concert/c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 scale=0.001 0.001 0.001
- link J6_A_stator: geometry collision mesh filename=package://concert_resources/models/modular/meshes/concert/s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 scale=0.001 0.001 0.001; visual mesh filename=package://concert_resources/models/modular/meshes/concert/c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 scale=0.001 0.001 0.001
- link L_1_A: geometry collision mesh filename=package://concert_resources/models/modular/meshes/concert/s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 scale=0.001 0.001 0.001; visual mesh filename=package://concert_resources/models/modular/meshes/concert/c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 scale=0.001 0.001 0.001
- link L_2_A: geometry collision mesh filename=package://concert_resources/models/modular/meshes/concert/s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 scale=0.001 0.001 0.001; visual mesh filename=package://concert_resources/models/modular/meshes/concert/c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 scale=0.001 0.001 0.001
- link L_3_A: geometry collision mesh filename=package://concert_resources/models/modular/meshes/concert/s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 scale=0.001 0.001 0.001; visual mesh filename=package://concert_resources/models/modular/meshes/concert/c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 scale=0.001 0.001 0.001
- link L_4_A: geometry collision mesh filename=package://concert_resources/models/modular/meshes/concert/s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 scale=0.001 0.001 0.001; visual mesh filename=package://concert_resources/models/modular/meshes/concert/c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 scale=0.001 0.001 0.001
- link L_5_A: geometry collision mesh filename=package://concert_resources/models/modular/meshes/concert/s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 scale=0.001 0.001 0.001; visual mesh filename=package://concert_resources/models/modular/meshes/concert/c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 scale=0.001 0.001 0.001
- link L_6_A: geometry collision mesh filename=package://concert_resources/models/modular/meshes/concert/s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 scale=0.001 0.001 0.001; visual mesh filename=package://concert_resources/models/modular/meshes/concert/c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 scale=0.001 0.001 0.001
- link dagana_A_bottom_link: geometry collision mesh filename=package://dagana_urdf/meshes/dg0002-ch.stl scale=0.001 0.001 0.001; visual mesh filename=package://dagana_urdf/meshes/dg0002.stl scale=0.001 0.001 0.001
- link dagana_A_top_link: geometry collision mesh filename=package://dagana_urdf/meshes/dg0001-simplified_v2.stl scale=0.001 0.001 0.001; visual mesh filename=package://dagana_urdf/meshes/dg0001-simplified.stl scale=0.001 0.001 0.001
